Commit message: works

File: urdf/three_dof.urdf (robot description, URDF)
Before this commit: robot simple_robot, 5 links, 4 joints
Links:
- added link ballpoint_link
- link ball_link: mass None -> 5; geometry collision sphere radius=0.02; visual sphere radius=0.02
- link base_link: geometry visual box size=0.5 0.5 0.1
- link column_link: geometry visual cylinder length=0.5 radius=0.02
- link plate_link: geometry collision cylinder length=0.02 radius=0.35; visual cylinder length=0.02 radius=0.35
Joints:
- removed joint column_to_point
- removed joint plate_to_ball
- removed joint point_to_plate
- added joint ballx: type prismatic, parent plate_link, child ballpoint_link, origin xyz=0 0 0.02 rpy=0 0 0, axis 1 0 0, limit lower=-0.35 upper=0.35 effort=1000.0 velocity=0.5
- added joint bally: type prismatic, parent ballpoint_link, child ball_link, origin xyz=0 0 0 rpy=0 0 0, axis 0 1 0, limit lower=-0.35 upper=0.35 effort=1000.0 velocity=0.5
- added joint pitch: type revolute, parent column_link, child point_link, origin xyz=0 0 0.25 rpy=0 0 0, axis 1 0 0, limit lower=-0.8 upper=0.8 effort=10 velocity=1
- added joint roll: type revolute, parent point_link, child plate_link, origin xyz=0 0 0 rpy=0 0 0, axis 0 1 0, limit lower=-0.8 upper=0.8 effort=10 velocity=1
- joint base_to_column: origin xyz=0 0 0.05 rpy=0 0 0 -> xyz=0 0 0.25 rpy=0 0 0

Commit message: clean code

File: urdf/three_dof.urdf (robot description, URDF)
Before this commit: robot simple_robot, 6 links, 5 joints
Links:
- link ballpoint_link: mass None -> 0.1
- link base_link: mass None -> 1; geometry collision box size=0.5 0.5 0.1; visual box size=0.5 0.5 0.1
- link column_link: mass None -> 0.5; geometry collision cylinder length=0.5 radius=0.02; visual cylinder length=0.5 radius=0.02
- link plate_link: mass None -> 0.5
- link point_link: mass None -> 0.1
